File: Hardware/ArtNetNode/ArtNetNode.kicad_pcb (KiCad board)
At the start: 2 copper layers, 100 x 100 mm, 136 parts, among them IC1 ISO1641BDR, IC2 ISO1641BDR, IC3 ISO1641BDR, IC4 ISO1641BDR, IC5 ISO1641BDR, IC6 ISO1641BDR, IC7 ISO1641BDR, IC8 ISO1641BDR, J1 B3B-XH-A, J2 B3B-XH-A, J3 B3B-XH-A, J4 B3B-XH-A, J5 B3B-XH-A, J6 B3B-XH-A, J7 B3B-XH-A, J8 B3B-XH-A, U1 MAX485E, U2 MAX485E, U3 MAX485E, U4 MAX485E, U5 MAX485E, U6 MAX485E, U7 MAX485E, U8 MAX485E

Commit message: finished dmx interfaces
Parts:
- removed C32, C34, C35, C36, C37, C38, C40, C41, C42, C43, C44, C46, C47, C48: 2u2/6V3, Capacitor_SMD:C_0603_1608Metric
- removed C33, C39, C45: 470p/2kV, Capacitor_SMD:C_1206_3216Metric
- removed IC1, IC2, IC3, IC4, IC5, IC6, IC7, IC8: ISO1641BDR, SamacSys_Parts:SOIC127P600X175-8N
- removed J6, J7, J8: B3B-XH-A, SamacSys_Parts:B3B-XH-A
- removed PS5, PS6, PS7, PS8: 1S4E_0505S1.5U, SamacSys_Parts:1S4E_0505S15U
- added R57: 0, Resistor_SMD:R_0603_1608Metric, F.Cu at (125.2, 68.5)
- added R58: 49R9, Resistor_SMD:R_0603_1608Metric, F.Cu at (125.2, 71.0)
- added R59: 49R9, Resistor_SMD:R_0603_1608Metric, F.Cu at (129.2, 53.4)
- added R60: 49R9, Resistor_SMD:R_0603_1608Metric, F.Cu at (129.2, 55.9)
- added R61: 49R9, Resistor_SMD:R_0603_1608Metric, F.Cu at (129.2, 58.4)
- added R62: 10R, Resistor_SMD:R_0603_1608Metric, F.Cu at (129.2, 60.9)
- added R63: 0, Resistor_SMD:R_0603_1608Metric, B.Cu at (84.6, 5.80)
- added R64: 0, Resistor_SMD:R_0603_1608Metric, B.Cu at (84.6, 44.8)
- added R65: 0, Resistor_SMD:R_0603_1608Metric, B.Cu at (84.6, 31.8)
- added R66: 0, Resistor_SMD:R_0603_1608Metric, B.Cu at (84.6, 18.8)
- added R67: 0, Resistor_SMD:R_0603_1608Metric, B.Cu at (84.6, 2.60)
- added R68: 0, Resistor_SMD:R_0603_1608Metric, B.Cu at (84.6, 41.6)
- added R69: 0, Resistor_SMD:R_0603_1608Metric, B.Cu at (84.6, 28.6)
- added R70: 0, Resistor_SMD:R_0603_1608Metric, B.Cu at (84.6, 15.6)
- added R71: 10k, Resistor_SMD:R_0603_1608Metric, F.Cu at (69.8, 2.60)
- added R72: 10k, Resistor_SMD:R_0603_1608Metric, F.Cu at (69.8, 41.6)
- added R73: 10k, Resistor_SMD:R_0603_1608Metric, F.Cu at (69.8, 28.6)
- added R74: 10k, Resistor_SMD:R_0603_1608Metric, F.Cu at (69.8, 15.6)
- added U10: LTV-356T, Package_SO:SO-4_4.4x3.6mm_P2.54mm, F.Cu at (76.6, 28.2)
- added U11: LTV-356T, Package_SO:SO-4_4.4x3.6mm_P2.54mm, B.Cu at (76.6, 28.6)
- added U12: LTV-356T, Package_SO:SO-4_4.4x3.6mm_P2.54mm, B.Cu at (76.6, 32.8)
- added U13: MAX485E, Package_SO:SOIC-8_3.9x4.9mm_P1.27mm, F.Cu at (87.2, 31.8)
- added U14: LTV-356T, Package_SO:SO-4_4.4x3.6mm_P2.54mm, F.Cu at (76.6, 15.2)
- added U15: LTV-356T, Package_SO:SO-4_4.4x3.6mm_P2.54mm, B.Cu at (76.6, 15.6)
- added U16: LTV-356T, Package_SO:SO-4_4.4x3.6mm_P2.54mm, B.Cu at (76.6, 19.8)
- added U17: MAX485E, Package_SO:SOIC-8_3.9x4.9mm_P1.27mm, F.Cu at (87.2, 18.8)
- added U18: W5500, Package_QFP:LQFP-48_7x7mm_P0.5mm, F.Cu at (227.3, 22.8)
- added U9: MAX485E, Package_SO:SOIC-8_3.9x4.9mm_P1.27mm, F.Cu at (87.2, 44.8)
- C10, C14, C2, C6: value 2u2/6V3 -> 470p/2kV; footprint Capacitor_SMD:C_0603_1608Metric -> Capacitor_SMD:C_1206_3216Metric; moved to B.Cu
- C15, C3, C9: value 470p/2kV -> 2u2/6V3; footprint Capacitor_SMD:C_1206_3216Metric -> Capacitor_SMD:C_0603_1608Metric
- C17: value 2u2/6V3 -> 10u/6V3; footprint Capacitor_SMD:C_0603_1608Metric -> Capacitor_SMD:C_0805_2012Metric
- C18, C19, C20, C22, C23, C24, C25, C26: value 2u2/6V3 -> 0u1/6V3
- C21: value 470p/2kV -> 0u1/6V3; footprint Capacitor_SMD:C_1206_3216Metric -> Capacitor_SMD:C_0603_1608Metric
- C27: value 470p/2kV -> 10u/6V3; footprint Capacitor_SMD:C_1206_3216Metric -> Capacitor_SMD:C_0603_1608Metric
- C28: value 2u2/6V3 -> 10n/63V
- C29: value 2u2/6V3 -> 22n/62V
- C30, C31: value 2u2/6V3 -> 6n8/63V
- J2: value B3B-XH-A -> ARJM11D7-104-AB-EW2; footprint SamacSys_Parts:B3B-XH-A -> SamacSys_Parts:ARJM11D7104ABEW2
- R1, R2, R25, R31, R32, R37, R38, R43, R44, R45, R8, R9: moved to B.Cu
- R10, R22, R24, R36, R46: value 10k -> 100k
- R11, R23: value 10k -> 120
- R13, R20: value 120 -> 10k; moved to B.Cu
- R14, R19, R21, R26, R33, R7: value 100k -> 10k; moved to B.Cu
- R15, R16, R3, R39, R4: value 10k -> 100; moved to B.Cu
- R18, R30: value 10k -> 100
- R27: value 120 -> 100; moved to B.Cu
- R28, R40: value 100k -> 100; moved to B.Cu
- R34, R48: value 120 -> 100k
- R35, R47: value 100k -> 120
- R41: value 120 -> 10k
- R42: value 100k -> 100
- R49: value 100k -> 12k4
- R5: value 100k -> 10k
- R50, R51, R52, R53: value 10k -> 330
- R54, R56: value 100k -> 0
- R55: value 120 -> 0
- R6: value 120 -> 100
- U1, U6: value MAX485E -> LTV-356T; footprint Package_SO:SOIC-8_3.9x4.9mm_P1.27mm -> Package_SO:SO-4_4.4x3.6mm_P2.54mm
- U2, U3, U7, U8: value MAX485E -> LTV-356T; footprint Package_SO:SOIC-8_3.9x4.9mm_P1.27mm -> Package_SO:SO-4_4.4x3.6mm_P2.54mm; moved to B.Cu
- U5: value MAX485E -> RP2040; footprint Package_SO:SOIC-8_3.9x4.9mm_P1.27mm -> Package_DFN_QFN:QFN-56-1EP_7x7mm_P0.4mm_EP3.2x3.2mm
- moved J2 202.4 mm to (137.1, -80.9)
- moved U2 174.8 mm to (76.6, 2.60)
- moved U5 167.6 mm to (224.4, 94.6)
- moved U4 167.3 mm to (87.2, 5.80)
- moved PS4 164.4 mm to (72.8, 22.7)
- moved J4 160.5 mm to (96.0, 34.3)
- moved R29 159.5 mm to (69.8, 27.0), turned to 180 degrees
- moved R28 159.1 mm to (69.8, 29.8), turned to 180 degrees
- moved R26 158.8 mm to (69.8, 27.4)
- moved R27 158.4 mm to (69.8, 34.0), turned to 180 degrees
- moved R25 158.2 mm to (69.8, 31.6)
- moved U1 154.1 mm to (76.6, 2.20), turned to 180 degrees
- moved C10 150.8 mm to (76.6, 37.8), turned to 0 degrees
- moved U7 150.4 mm to (76.6, 41.6)
- moved C9 149.3 mm to (74.2, 37.8), turned to 180 degrees
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Connections:
- C10 pad 1: /DMX_DRIVER1/ISO_5V -> GND
- C10 pad 2: /DMX_DRIVER1/ISO_GND -> /DMX_DRIVER2/ISO_GND
- C11 pad 1: /DMX_DRIVER1/ISO_5V -> /DMX_DRIVER2/ISO_5V
- C11 pad 2: /DMX_DRIVER1/ISO_GND -> /DMX_DRIVER2/ISO_GND
- C12 pad 1: /DMX_DRIVER1/ISO_5V -> /DMX_DRIVER2/ISO_5V
- C12 pad 2: /DMX_DRIVER1/ISO_GND -> /DMX_DRIVER2/ISO_GND
- C14 pad 1: +5V -> GND
- C14 pad 2: GND -> /DMX_DRIVER3/ISO_GND
- C15 pad 1: GND -> /DMX_DRIVER3/ISO_5V
- C15 pad 2: /DMX_DRIVER2/ISO_GND -> /DMX_DRIVER3/ISO_GND
- C16 pad 1: /DMX_DRIVER2/ISO_5V -> /DMX_DRIVER3/ISO_5V
- C16 pad 2: /DMX_DRIVER2/ISO_GND -> /DMX_DRIVER3/ISO_GND
- C17 pad 1: /DMX_DRIVER2/ISO_5V -> +3V3
- C17 pad 2: /DMX_DRIVER2/ISO_GND -> GND
- C18 pad 1: /DMX_DRIVER2/ISO_5V -> +3V3
- C18 pad 2: /DMX_DRIVER2/ISO_GND -> GND
- C19 pad 1: +5V -> +3V3
- C2 pad 1: +5V -> GND
- C2 pad 2: GND -> /DMX_DRIVER0/ISO_GND
- C20 pad 1: +5V -> Net-(U18-1V2O)
- C21 pad 1: GND -> +3V3
- C21 pad 2: /DMX_DRIVER3/ISO_GND -> GND
- C22 pad 1: /DMX_DRIVER3/ISO_5V -> Net-(U18-TOCAP)
- C22 pad 2: /DMX_DRIVER3/ISO_GND -> GND
- C23 pad 1: /DMX_DRIVER3/ISO_5V -> +3V3
- C23 pad 2: /DMX_DRIVER3/ISO_GND -> GND
- C24 pad 1: /DMX_DRIVER3/ISO_5V -> +3V3
- C24 pad 2: /DMX_DRIVER3/ISO_GND -> GND
- C25 pad 1: +5V -> +3V3
- C26 pad 1: +5V -> +3V3
- C27 pad 1: GND -> +3V3
- C27 pad 2: /DMX_DRIVER4/ISO_GND -> GND
- C28 pad 1: /DMX_DRIVER4/ISO_5V -> /ETHERNET/PHY/RCT
- C28 pad 2: /DMX_DRIVER4/ISO_GND -> GND
- C29 pad 1: /DMX_DRIVER4/ISO_5V -> /ETHERNET/PHY/TCT
- C29 pad 2: /DMX_DRIVER4/ISO_GND -> GND
- C3 pad 1: GND -> /DMX_DRIVER0/ISO_5V
- C30 pad 1: /DMX_DRIVER4/ISO_5V -> /ETHERNET/PHY/RD-
- C30 pad 2: /DMX_DRIVER4/ISO_GND -> Net-(C30-Pad2)
- C31 pad 1: +5V -> Net-(C31-Pad1)
- C31 pad 2: GND -> /ETHERNET/PHY/RD+
- C5 pad 1: /DMX_DRIVER0/ISO_5V -> +5V
- C5 pad 2: /DMX_DRIVER0/ISO_GND -> GND
- C6 pad 1: /DMX_DRIVER0/ISO_5V -> GND
- C6 pad 2: /DMX_DRIVER0/ISO_GND -> /DMX_DRIVER1/ISO_GND
- C7 pad 1: +5V -> /DMX_DRIVER1/ISO_5V
- C7 pad 2: GND -> /DMX_DRIVER1/ISO_GND
- C8 pad 1: +5V -> /DMX_DRIVER1/ISO_5V
- C8 pad 2: GND -> /DMX_DRIVER1/ISO_GND
- C9 pad 1: GND -> +5V
- C9 pad 2: /DMX_DRIVER1/ISO_GND -> GND
- J1 pad 1: Net-(U1-A) -> Net-(U4-A)
- J1 pad 3: Net-(U1-B) -> Net-(U4-B)
- J2 pad 1: Net-(U2-A) -> unconnected-(J2-TD+-Pad1)
- J2 pad 2: /DMX_DRIVER1/ISO_GND -> unconnected-(J2-TD--Pad2)
- J2 pad 3: Net-(U2-B) -> unconnected-(J2-RD+-Pad3)
- J3 pad 1: Net-(U3-A) -> Net-(U9-A)
- J3 pad 2: /DMX_DRIVER2/ISO_GND -> /DMX_DRIVER1/ISO_GND
- J3 pad 3: Net-(U3-B) -> Net-(U9-B)
- J4 pad 1: Net-(U4-A) -> Net-(U13-A)
- J4 pad 2: /DMX_DRIVER3/ISO_GND -> /DMX_DRIVER2/ISO_GND
- J4 pad 3: Net-(U4-B) -> Net-(U13-B)
- J5 pad 1: Net-(U5-A) -> Net-(U17-A)
- J5 pad 2: /DMX_DRIVER4/ISO_GND -> /DMX_DRIVER3/ISO_GND
- J5 pad 3: Net-(U5-B) -> Net-(U17-B)
- R1 pad 1: +5V -> +3.3V
- R1 pad 2: /DMX_DRIVER0/DMX_DATA -> /DMX_DRIVER0/TX
- R10 pad 1: /DMX_DRIVER1/ISO_5V -> /DMX_DRIVER0/ISO_5V
- R10 pad 2: Net-(IC2-SCL2) -> Net-(U4-A)
- R11 pad 1: /DMX_DRIVER1/ISO_5V -> Net-(U4-A)
- R11 pad 2: Net-(IC2-SDA2) -> Net-(U4-B)
- R12 pad 1: /DMX_DRIVER1/ISO_5V -> Net-(U4-B)
- R12 pad 2: Net-(U2-A) -> /DMX_DRIVER0/ISO_GND
- R13 pad 1: Net-(U2-A) -> +3.3V
- R13 pad 2: Net-(U2-B) -> /DMX_DRIVER1/TX
- R14 pad 1: Net-(U2-B) -> +3.3V
- R14 pad 2: /DMX_DRIVER1/ISO_GND -> /DMX_DRIVER1/DIR
- R15 pad 1: +5V -> Net-(R15-Pad1)
- R15 pad 2: /DMX_DRIVER2/DMX_DATA -> +3.3V
- R16 pad 1: +5V -> Net-(R16-Pad1)
- R16 pad 2: /DMX_DRIVER2/DMX_DIR -> +3.3V
- R17 pad 1: /DMX_DRIVER2/ISO_5V -> /DMX_DRIVER1/RX
- R17 pad 2: Net-(IC3-SCL2) -> GND
- R18 pad 1: /DMX_DRIVER2/ISO_5V -> Net-(R18-Pad1)
- R18 pad 2: Net-(IC3-SDA2) -> Net-(U9-RO)
- R19 pad 1: /DMX_DRIVER2/ISO_5V -> /DMX_DRIVER1/ISO_5V
- R19 pad 2: Net-(U3-A) -> Net-(U9-DI)
- R2 pad 1: +5V -> +3.3V
- R2 pad 2: /DMX_DRIVER0/DMX_DIR -> /DMX_DRIVER0/DIR
- R20 pad 1: Net-(U3-A) -> /DMX_DRIVER1/ISO_5V
- R20 pad 2: Net-(U3-B) -> Net-(U9-DE)
- R21 pad 1: Net-(U3-B) -> /DMX_DRIVER1/ISO_5V
- R21 pad 2: /DMX_DRIVER2/ISO_GND -> Net-(U9-RO)
- R22 pad 1: +5V -> /DMX_DRIVER1/ISO_5V
- R22 pad 2: /DMX_DRIVER3/DMX_DATA -> Net-(U9-A)
- R23 pad 1: +5V -> Net-(U9-A)
- R23 pad 2: /DMX_DRIVER3/DMX_DIR -> Net-(U9-B)
- R24 pad 1: /DMX_DRIVER3/ISO_5V -> Net-(U9-B)
- R24 pad 2: Net-(IC4-SCL2) -> /DMX_DRIVER1/ISO_GND
- R25 pad 1: /DMX_DRIVER3/ISO_5V -> +3.3V
- R25 pad 2: Net-(IC4-SDA2) -> /DMX_DRIVER2/TX
- R26 pad 1: /DMX_DRIVER3/ISO_5V -> +3.3V
- R26 pad 2: Net-(U4-A) -> /DMX_DRIVER2/DIR
- R27 pad 1: Net-(U4-A) -> Net-(R27-Pad1)
- R27 pad 2: Net-(U4-B) -> +3.3V
- R28 pad 1: Net-(U4-B) -> Net-(R28-Pad1)
- R28 pad 2: /DMX_DRIVER3/ISO_GND -> +3.3V
- R29 pad 1: +5V -> /DMX_DRIVER2/RX
- R29 pad 2: /DMX_DRIVER4/DMX_DATA -> GND
- R3 pad 1: /DMX_DRIVER0/ISO_5V -> Net-(R3-Pad1)
- R3 pad 2: Net-(IC1-SCL2) -> +3.3V
- R30 pad 1: +5V -> Net-(R30-Pad1)
- R30 pad 2: /DMX_DRIVER4/DMX_DIR -> Net-(U13-RO)
- R31 pad 1: /DMX_DRIVER4/ISO_5V -> /DMX_DRIVER2/ISO_5V
- R31 pad 2: Net-(IC5-SCL2) -> Net-(U13-DI)
- R32 pad 1: /DMX_DRIVER4/ISO_5V -> /DMX_DRIVER2/ISO_5V
- R32 pad 2: Net-(IC5-SDA2) -> Net-(U13-DE)
- R33 pad 1: /DMX_DRIVER4/ISO_5V -> /DMX_DRIVER2/ISO_5V
- R33 pad 2: Net-(U5-A) -> Net-(U13-RO)
- R34 pad 1: Net-(U5-A) -> /DMX_DRIVER2/ISO_5V
- R34 pad 2: Net-(U5-B) -> Net-(U13-A)
- R35 pad 1: Net-(U5-B) -> Net-(U13-A)
- R35 pad 2: /DMX_DRIVER4/ISO_GND -> Net-(U13-B)
- R36 pad 1: +5V -> Net-(U13-B)
- R36 pad 2: /DMX_DRIVER5/DMX_DATA -> /DMX_DRIVER2/ISO_GND
- R37 pad 1: +5V -> +3.3V
- R37 pad 2: /DMX_DRIVER5/DMX_DIR -> /DMX_DRIVER3/TX
- R38 pad 1: /DMX_DRIVER5/ISO_5V -> +3.3V
- R38 pad 2: Net-(IC6-SCL2) -> /DMX_DRIVER3/DIR
- R39 pad 1: /DMX_DRIVER5/ISO_5V -> Net-(R39-Pad1)
- R39 pad 2: Net-(IC6-SDA2) -> +3.3V
- R4 pad 1: /DMX_DRIVER0/ISO_5V -> Net-(R4-Pad1)
- R4 pad 2: Net-(IC1-SDA2) -> +3.3V
- R40 pad 1: /DMX_DRIVER5/ISO_5V -> Net-(R40-Pad1)
- R40 pad 2: Net-(U6-A) -> +3.3V
- R41 pad 1: Net-(U6-A) -> /DMX_DRIVER3/RX
- R41 pad 2: Net-(U6-B) -> GND
- R42 pad 1: Net-(U6-B) -> Net-(R42-Pad1)
- R42 pad 2: /DMX_DRIVER5/ISO_GND -> Net-(U17-RO)
- R43 pad 1: +5V -> /DMX_DRIVER3/ISO_5V
- R43 pad 2: /DMX_DRIVER6/DMX_DATA -> Net-(U17-DI)
- R44 pad 1: +5V -> /DMX_DRIVER3/ISO_5V
- R44 pad 2: /DMX_DRIVER6/DMX_DIR -> Net-(U17-DE)
- R45 pad 1: /DMX_DRIVER6/ISO_5V -> /DMX_DRIVER3/ISO_5V
- R45 pad 2: Net-(IC7-SCL2) -> Net-(U17-RO)
- R46 pad 1: /DMX_DRIVER6/ISO_5V -> /DMX_DRIVER3/ISO_5V
- R46 pad 2: Net-(IC7-SDA2) -> Net-(U17-A)
- R47 pad 1: /DMX_DRIVER6/ISO_5V -> Net-(U17-A)
- R47 pad 2: Net-(U7-A) -> Net-(U17-B)
- R48 pad 1: Net-(U7-A) -> Net-(U17-B)
- R48 pad 2: Net-(U7-B) -> /DMX_DRIVER3/ISO_GND
- R49 pad 1: Net-(U7-B) -> GND
- R49 pad 2: /DMX_DRIVER6/ISO_GND -> Net-(U18-EXRES1)
- R5 pad 1: /DMX_DRIVER0/ISO_5V -> /DMX_DRIVER0/RX
- R5 pad 2: Net-(U1-A) -> GND
- R50 pad 1: +5V -> Net-(U18-SPDLED)
- R50 pad 2: /DMX_DRIVER7/DMX_DATA -> /ETHERNET/PHY/SPDLED
- R51 pad 1: +5V -> Net-(U18-LINKLED)
- R51 pad 2: /DMX_DRIVER7/DMX_DIR -> /ETHERNET/PHY/LINKLED
- R52 pad 1: /DMX_DRIVER7/ISO_5V -> Net-(U18-DUPLED)
- R52 pad 2: Net-(IC8-SCL2) -> /ETHERNET/PHY/DUPLED
- R53 pad 1: /DMX_DRIVER7/ISO_5V -> Net-(U18-ACTLED)
- R53 pad 2: Net-(IC8-SDA2) -> /ETHERNET/PHY/ACTLED
- R54 pad 1: /DMX_DRIVER7/ISO_5V -> /ETHERNET/PHY/TX_N
- R54 pad 2: Net-(U8-A) -> /ETHERNET/PHY/TCT
- R55 pad 1: Net-(U8-A) -> /ETHERNET/PHY/TX_P
- R55 pad 2: Net-(U8-B) -> /ETHERNET/PHY/TCT
- R56 pad 1: Net-(U8-B) -> /ETHERNET/PHY/RX_N
- R56 pad 2: /DMX_DRIVER7/ISO_GND -> Net-(C30-Pad2)
- R6 pad 1: Net-(U1-A) -> Net-(R6-Pad1)
- R6 pad 2: Net-(U1-B) -> Net-(U4-RO)
- R7 pad 1: Net-(U1-B) -> /DMX_DRIVER0/ISO_5V
- R7 pad 2: /DMX_DRIVER0/ISO_GND -> Net-(U4-DI)
- R8 pad 1: +5V -> /DMX_DRIVER0/ISO_5V
- R8 pad 2: /DMX_DRIVER1/DMX_DATA -> Net-(U4-DE)
- R9 pad 1: +5V -> /DMX_DRIVER0/ISO_5V
- R9 pad 2: /DMX_DRIVER1/DMX_DIR -> Net-(U4-RO)
- U1 pad 1: Net-(IC1-SDA2) -> Net-(R6-Pad1)
- U1 pad 2: Net-(IC1-SCL2) -> /DMX_DRIVER0/ISO_GND
- U1 pad 3: Net-(IC1-SCL2) -> /DMX_DRIVER0/RX
- U1 pad 4: Net-(IC1-SDA2) -> +3.3V
- U2 pad 1: Net-(IC2-SDA2) -> Net-(R4-Pad1)
- U2 pad 2: Net-(IC2-SCL2) -> /DMX_DRIVER0/DIR
- U2 pad 3: Net-(IC2-SCL2) -> /DMX_DRIVER0/ISO_GND
- U2 pad 4: Net-(IC2-SDA2) -> Net-(U4-DE)
- U3 pad 1: Net-(IC3-SDA2) -> Net-(R3-Pad1)
- U3 pad 2: Net-(IC3-SCL2) -> /DMX_DRIVER0/TX
- U3 pad 3: Net-(IC3-SCL2) -> /DMX_DRIVER0/ISO_GND
- U3 pad 4: Net-(IC3-SDA2) -> Net-(U4-DI)
- U4 pad 1: Net-(IC4-SDA2) -> Net-(U4-RO)
- U4 pad 2: Net-(IC4-SCL2) -> Net-(U4-~{RE})
- U4 pad 3: Net-(IC4-SCL2) -> Net-(U4-DE)
- U4 pad 4: Net-(IC4-SDA2) -> Net-(U4-DI)
- U4 pad 5: /DMX_DRIVER3/ISO_GND -> /DMX_DRIVER0/ISO_GND
- U4 pad 8: /DMX_DRIVER3/ISO_5V -> /DMX_DRIVER0/ISO_5V
- U5 pad 1: Net-(IC5-SDA2) -> Net-(U5-IOVDD-Pad1)
- U5 pad 2: Net-(IC5-SCL2) -> unconnected-(U5-GPIO0-Pad2)
- U5 pad 3: Net-(IC5-SCL2) -> unconnected-(U5-GPIO1-Pad3)
- U5 pad 4: Net-(IC5-SDA2) -> unconnected-(U5-GPIO2-Pad4)
- U5 pad 5: /DMX_DRIVER4/ISO_GND -> unconnected-(U5-GPIO3-Pad5)
- U5 pad 6: Net-(U5-A) -> unconnected-(U5-GPIO4-Pad6)
- U5 pad 7: Net-(U5-B) -> unconnected-(U5-GPIO5-Pad7)
- U5 pad 8: /DMX_DRIVER4/ISO_5V -> unconnected-(U5-GPIO6-Pad8)
- U6 pad 1: Net-(IC6-SDA2) -> Net-(R18-Pad1)
- U6 pad 2: Net-(IC6-SCL2) -> /DMX_DRIVER1/ISO_GND
- U6 pad 3: Net-(IC6-SCL2) -> /DMX_DRIVER1/RX
- U6 pad 4: Net-(IC6-SDA2) -> +3.3V
- U7 pad 1: Net-(IC7-SDA2) -> Net-(R16-Pad1)
- U7 pad 2: Net-(IC7-SCL2) -> /DMX_DRIVER1/DIR
- U7 pad 3: Net-(IC7-SCL2) -> /DMX_DRIVER1/ISO_GND
- U7 pad 4: Net-(IC7-SDA2) -> Net-(U9-DE)
- U8 pad 1: Net-(IC8-SDA2) -> Net-(R15-Pad1)
- U8 pad 2: Net-(IC8-SCL2) -> /DMX_DRIVER1/TX
- U8 pad 3: Net-(IC8-SCL2) -> /DMX_DRIVER1/ISO_GND
- U8 pad 4: Net-(IC8-SDA2) -> Net-(U9-DI)
