File: Hardware/ArtNetNode/ArtNetNode.kicad_sch (KiCad schematic)
At the start: 0 parts

Commit message: finished dmx interfaces
Other:
- removed sheet DMX_DRIVER4
- removed sheet DMX_DRIVER5
- removed sheet DMX_DRIVER6
- removed sheet DMX_DRIVER7
- sheet DMX_DRIVER0 ports: added DIR, RX, TX; removed DMX_DATA, DMX_DIR
- sheet DMX_DRIVER1 ports: added DIR, RX, TX; removed DMX_DATA, DMX_DIR
- sheet DMX_DRIVER2 ports: added DIR, RX, TX; removed DMX_DATA, DMX_DIR
- sheet DMX_DRIVER3 ports: added DIR, RX, TX; removed DMX_DATA, DMX_DIR
