File: Hardware/ArtNetNode/W5500.kicad_sch (KiCad schematic)
At the start: 30 parts, among them U10 W5500

Commit message: finished dmx interfaces
Parts:
- C17: renamed from C57; footprint (none) -> Capacitor_SMD:C_0805_2012Metric
- C18: renamed from C56; footprint (none) -> Capacitor_SMD:C_0603_1608Metric
- C19: renamed from C49; footprint (none) -> Capacitor_SMD:C_0603_1608Metric
- C20: renamed from C63; footprint (none) -> Capacitor_SMD:C_0603_1608Metric
- C21: renamed from C50; footprint (none) -> Capacitor_SMD:C_0603_1608Metric
- C22: renamed from C62; footprint (none) -> Capacitor_SMD:C_0603_1608Metric
- C23: renamed from C51; footprint (none) -> Capacitor_SMD:C_0603_1608Metric
- C24: renamed from C52; footprint (none) -> Capacitor_SMD:C_0603_1608Metric
- C25: renamed from C53; footprint (none) -> Capacitor_SMD:C_0603_1608Metric
- C26: renamed from C54; footprint (none) -> Capacitor_SMD:C_0603_1608Metric
- C27: renamed from C55; footprint (none) -> Capacitor_SMD:C_0603_1608Metric
- C28: renamed from C61; footprint (none) -> Capacitor_SMD:C_0603_1608Metric
- C29: renamed from C58; footprint (none) -> Capacitor_SMD:C_0603_1608Metric
- C30: renamed from C59; footprint (none) -> Capacitor_SMD:C_0603_1608Metric
- C31: renamed from C60; footprint (none) -> Capacitor_SMD:C_0603_1608Metric
- R49: renamed from R70; footprint (none) -> Resistor_SMD:R_0603_1608Metric
- R50: renamed from R66; footprint (none) -> Resistor_SMD:R_0603_1608Metric
- R51: renamed from R67; footprint (none) -> Resistor_SMD:R_0603_1608Metric
- R52: renamed from R68; footprint (none) -> Resistor_SMD:R_0603_1608Metric
- R53: renamed from R69; footprint (none) -> Resistor_SMD:R_0603_1608Metric
- R54: renamed from R57; footprint (none) -> Resistor_SMD:R_0603_1608Metric
- R55: renamed from R58; footprint (none) -> Resistor_SMD:R_0603_1608Metric
- R56: renamed from R59; footprint (none) -> Resistor_SMD:R_0603_1608Metric
- R57: renamed from R60; footprint (none) -> Resistor_SMD:R_0603_1608Metric
- R58: renamed from R61; footprint (none) -> Resistor_SMD:R_0603_1608Metric
- R59: renamed from R64; footprint (none) -> Resistor_SMD:R_0603_1608Metric
- R60: renamed from R62; footprint (none) -> Resistor_SMD:R_0603_1608Metric
- R61: renamed from R65; footprint (none) -> Resistor_SMD:R_0603_1608Metric
- R62: renamed from R63; footprint (none) -> Resistor_SMD:R_0603_1608Metric
- renumbered U10 to U18
