File: Hardware/ArtNetNode/ethernet.kicad_sch (KiCad schematic)
At the start: 0 parts

Commit message: added ethernet
Parts:
- added J9: ARJM11D7-104-AB-EW2, ARJM11D7104ABEW2, symbol SamacSys_Parts:ARJM11D7-104-AB-EW2
Other:
- added sheet PHY (W5500.kicad_sch)

Commit message: finished dmx interfaces
Parts:
- J2: renamed from J9; footprint ARJM11D7104ABEW2 -> SamacSys_Parts:ARJM11D7104ABEW2
Changed lines of the file:
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@@
 		(dnp no)
 		(fields_autoplaced yes)
-		(property "Reference" "J9"
+		(property "Reference" "J2"
 			(at 313.69 124.46 0)
 			(effects
@@
 			)
 		)
-		(property "Footprint" "ARJM11D7104ABEW2"
+		(property "Footprint" "SamacSys_Parts:ARJM11D7104ABEW2"
 			(at 326.39 227 0)
 			(effects
@@
 			(project ""
 				(path "/5fe0a06d-00fb-4ef8-80af-4dd06c5496d9/d72acdc1-f649-4ceb-9a30-42cb477c4dd7"
-					(reference "J9")
+					(reference "J2")
 					(unit 1)
 				)
