File: Hardware/ArtNetNode/mcu.kicad_sch (KiCad schematic)
At the start: 0 parts

Commit message: added ethernet
Parts:
- added U9: RP2040, Package_DFN_QFN:QFN-56-1EP_7x7mm_P0.4mm_EP3.2x3.2mm, symbol MCU_RaspberryPi:RP2040
Connections:
- new net: U9.1 (IOVDD), U9.10 (IOVDD), U9.22 (IOVDD), U9.33 (IOVDD), U9.42 (IOVDD), U9.49 (IOVDD)
- new net: U9.23 (DVDD), U9.50 (DVDD)
Changed lines of the file:
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@@
 	(generator_version "8.0")
 	(paper "A3")
+	(symbol
+		(lib_id "MCU_RaspberryPi:RP2040")
+		(at 151.13 152.4 0)
+		(unit 1)
+		(exclude_from_sim no)
+		(in_bom yes)
+		(on_board yes)
+		(dnp no)
+		(fields_autoplaced yes)
+		(property "Reference" "U9"
+			(at 153.3241 196.85 0)
+			(effects
+				(font
+					(size 1.27 1.27)
+				)
+				(justify left)
+			)
+		)
+		(property "Value" "RP2040"
+			(at 153.3241 199.39 0)
+			(effects
+				(font
+					(size 1.27 1.27)
+				)
+				(justify left)
+			)
+		)
+		(property "Footprint" "Package_DFN_QFN:QFN-56-1EP_7x7mm_P0.4mm_EP3.2x3.2mm"
+			(at 151.13 152.4 0)
+			(effects
+				(font
+					(size 1.27 1.27)
+				)
+				(hide yes)
+			)
+		)
+		(property "Datasheet" "https://datasheets.raspberrypi.com/rp2040/rp2040-datasheet.pdf"
+			(at 151.13 152.4 0)
+			(effects
+				(font
+					(size 1.27 1.27)
+				)
+				(hide yes)
+			)
+		)
+		(property "Description" "A microcontroller by Raspberry Pi"
+			(at 151.13 152.4 0)
+			(effects
+				(font
+					(size 1.27 1.27)
+				)
+				(hide yes)
+			)
+		)
+		(pin "8"
+		)
+		(pin "6"
+		)
+		(pin "57"
+		)
+		(pin "9"
+		)
+		(pin "7"
+		)
+		(pin "56"
+		)
+		(pin "55"
+		)
+		(pin "2"
+		)
+		(pin "52"
+		)
+		(pin "16"
+		)
+		(pin "14"
+		)
+		(pin "1"
+		)
+		(pin "15"
+		)
+		(pin "22"
+		)
+		(pin "26"
+		)
+		(pin "12"
+		)
+		(pin "36"
+		)
+		(pin "40"
+		)
+		(pin "29"
+		)
+		(pin "42"
+		)
+		(pin "34"
+		)
+		(pin "30"
+		)
+		(pin "3"
+		)
+		(pin "27"
+		)
+		(pin "13"
+		)
+		(pin "24"
+		)
+		(pin "31"
+		)
+		(pin "35"
+		)
+		(pin "44"
+		)
+		(pin "45"
+		)
+		(pin "47"
+		)
+		(pin "23"
+		)
+		(pin "18"
+		)
+		(pin "48"
+		)
+		(pin "20"
+		)
+		(pin "11"
+		)
+		(pin "5"
+		)
+		(pin "17"
+		)
+		(pin "21"
+		)
+		(pin "37"
+		)
+		(pin "19"
+		)
+		(pin "51"
+		)
+		(pin "4"
+		)
+		(pin "53"
+		)
+		(pin "43"
+		)
+		(pin "46"
+		)
+		(pin "28"
+		)
+		(pin "32"
+		)
+		(pin "33"
+		)
+		(pin "38"
+		)
+		(pin "39"
+		)
+		(pin "50"
+		)
+		(pin "54"
+		)
+		(pin "10"
+		)
+		(pin "25"
+		)
+		(pin "41"
+		)
+		(pin "49"
+		)
+		(instances
+			(project ""
+				(path "/5fe0a06d-00fb-4ef8-80af-4dd06c5496d9/efc89bbc-2463-427a-9fa7-bd6145ec8808"
+					(reference "U9")
+					(unit 1)
+				)
+			)
+		)
+	)
 )

Commit message: finished dmx interfaces
Parts:
- renumbered U9 to U5
Other:
- moved on the sheet: U5
Changed lines of the file:
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@@
 	(symbol
 		(lib_id "MCU_RaspberryPi:RP2040")
-		(at 151.13 152.4 0)
+		(at 181.61 143.51 0)
 		(unit 1)
 		(exclude_from_sim no)
@@
 		(dnp no)
 		(fields_autoplaced yes)
-		(property "Reference" "U9"
-			(at 153.3241 196.85 0)
+		(property "Reference" "U5"
+			(at 183.8041 187.96 0)
 			(effects
 				(font
@@
 		)
 		(property "Value" "RP2040"
-			(at 153.3241 199.39 0)
+			(at 183.8041 190.5 0)
 			(effects
 				(font
@@
 		)
 		(property "Footprint" "Package_DFN_QFN:QFN-56-1EP_7x7mm_P0.4mm_EP3.2x3.2mm"
-			(at 151.13 152.4 0)
+			(at 181.61 143.51 0)
 			(effects
 				(font
@@
 		)
 		(property "Datasheet" "https://datasheets.raspberrypi.com/rp2040/rp2040-datasheet.pdf"
-			(at 151.13 152.4 0)
+			(at 181.61 143.51 0)
 			(effects
 				(font
@@
 		)
 		(property "Description" "A microcontroller by Raspberry Pi"
-			(at 151.13 152.4 0)
+			(at 181.61 143.51 0)
 			(effects
 				(font
@@
 			(project ""
 				(path "/5fe0a06d-00fb-4ef8-80af-4dd06c5496d9/efc89bbc-2463-427a-9fa7-bd6145ec8808"
-					(reference "U9")
+					(reference "U5")
 					(unit 1)
 				)
