File: hw_v1/ArtNetNode.kicad_pcb (KiCad board)
At the start: 4 copper layers, 100 x 100 mm, 67 parts, among them IC1 W25Q16JVSNIQ, IC2 RP2350B, J1 Conn_ARM_SWD_TagConnect_TC203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, J2 SM03B-SRSS-TB_LF__SN_, J3 SM03B-SRSS-TB_LF__SN_, J4 SM03B-SRSS-TB_LF__SN_, J5 SM03B-SRSS-TB_LF__SN_, SW1 SW_SPST, U1 ST485E, U2 ST485E, U3 ST485E, U4 ST485E, Y1 SiT1602AC-13-33E-12.000000

Commit message: started hardware
Parts:
- removed the D1 at (-31.3, 42.6)
- removed the D2 at (-31.3, 45.0)
- removed the D3 at (15.0, 8.00)
- removed the D4 at (30.0, 8.00)
- removed J2, J3, J4, J5: SM03B-SRSS-TB_LF__SN_, SamacSys_Parts:SM03BSRSSTBLFSN
- removed the R10 at (15.0, 11.5)
- removed the R7 at (-38.2, 28.7)
- removed the R8 at (-38.2, 31.2)
- removed the R9 at (12.0, 11.5)
- added C27: 1u/6V3, Capacitor_SMD:C_0603_1608Metric, F.Cu at (7.50, 13.5)
- added C28: 10u/6V3, Capacitor_SMD:C_0603_1608Metric, F.Cu at (18.2, 33.2)
- added C29: 10u/6V3, Capacitor_SMD:C_0603_1608Metric, F.Cu at (20.2, 13.5)
- added C30: 1u/6V3, Capacitor_SMD:C_0603_1608Metric, F.Cu at (19.2, 18.2)
- added C31: 10u/6V3, Capacitor_SMD:C_0603_1608Metric, F.Cu at (31.0, 33.2)
- added C32: 10u/6V3, Capacitor_SMD:C_0603_1608Metric, F.Cu at (32.0, 18.2)
- added C33: 1u/6V3, Capacitor_SMD:C_0603_1608Metric, F.Cu at (33.0, 13.5)
- added C34: 10u/6V3, Capacitor_SMD:C_0603_1608Metric, F.Cu at (43.8, 33.2)
- added C35: 10u/6V3, Capacitor_SMD:C_0603_1608Metric, F.Cu at (44.8, 18.2)
- added C36: 1u/6V3, Capacitor_SMD:C_0603_1608Metric, F.Cu at (45.8, 13.5)
- added C37: 10u/6V3, Capacitor_SMD:C_0603_1608Metric, F.Cu at (57.8, 33.2)
- added C38: 10u/6V3, Capacitor_SMD:C_0603_1608Metric, F.Cu at (58.8, 18.2)
- added C39: 1u/6V3, Capacitor_SMD:C_0603_1608Metric, F.Cu at (59.8, 13.5)
- added C40: 10u/6V3, Capacitor_SMD:C_0603_1608Metric, F.Cu at (70.5, 33.2)
- added C41: 10u/6V3, Capacitor_SMD:C_0603_1608Metric, F.Cu at (72.5, 13.5)
- added C42: 1u/6V3, Capacitor_SMD:C_0603_1608Metric, F.Cu at (71.5, 18.2)
- added C43: 10u/6V3, Capacitor_SMD:C_0603_1608Metric, F.Cu at (83.2, 33.2)
- added C44: 10u/6V3, Capacitor_SMD:C_0603_1608Metric, F.Cu at (85.2, 13.5)
- added C45: 1u/6V3, Capacitor_SMD:C_0603_1608Metric, F.Cu at (84.2, 18.2)
- added C46: 10u/6V3, Capacitor_SMD:C_0603_1608Metric, F.Cu at (96.0, 33.2)
- added C47: 10u/6V3, Capacitor_SMD:C_0603_1608Metric, F.Cu at (97.0, 18.2)
- added C48: 1u/6V3, Capacitor_SMD:C_0603_1608Metric, F.Cu at (98.0, 13.5)
- added C49: 10u/6V3, Capacitor_SMD:C_0603_1608Metric, F.Cu at (110.0, 33.2)
- added C50: 10u/6V3, Capacitor_SMD:C_0603_1608Metric, F.Cu at (112.0, 13.5)
- added C51: 1u/6V3, Capacitor_SMD:C_0603_1608Metric, F.Cu at (111.0, 18.2)
- added C52: 10u/6V3, Capacitor_SMD:C_0603_1608Metric, F.Cu at (122.8, 33.2)
- added C53: 10u/6V3, Capacitor_SMD:C_0603_1608Metric, F.Cu at (124.8, 13.5)
- added C54: 1u/6V3, Capacitor_SMD:C_0603_1608Metric, F.Cu at (123.8, 18.2)
- added C55: 10u/6V3, Capacitor_SMD:C_0603_1608Metric, F.Cu at (135.5, 33.2)
- added C56: 10u/6V3, Capacitor_SMD:C_0603_1608Metric, F.Cu at (137.5, 13.5)
- added C57: 1u/6V3, Capacitor_SMD:C_0603_1608Metric, F.Cu at (136.5, 18.2)
- added C58: 10u/6V3, Capacitor_SMD:C_0603_1608Metric, F.Cu at (148.2, 33.2)
- added C59: 10u/6V3, Capacitor_SMD:C_0603_1608Metric, F.Cu at (149.2, 18.2)
- added C60: 1u/6V3, Capacitor_SMD:C_0603_1608Metric, F.Cu at (150.2, 13.5)
- added C61: 10u/6V3, Capacitor_SMD:C_0603_1608Metric, F.Cu at (-17.3, 9.18)
- added C62: 10u/6V3, Capacitor_SMD:C_0603_1608Metric, F.Cu at (-17.3, 11.7)
- added C63: 10u/6V3, Capacitor_SMD:C_0603_1608Metric, F.Cu at (-17.3, 14.2)
- added C64: 10u/6V3, Capacitor_SMD:C_0603_1608Metric, F.Cu at (-17.3, 16.7)
- added C65: 10u/6V3, Capacitor_SMD:C_0603_1608Metric, F.Cu at (-17.3, 19.2)
- added C66: 10u/6V3, Capacitor_SMD:C_0603_1608Metric, F.Cu at (-17.3, 21.7)
- added D1: LED, LED_SMD:LED_0603_1608Metric, F.Cu at (-55.9, 13.5)
- added D1: PTVS5V0Z1USK, Diode_SMD:Nexperia_DSN1608-2_1.6x0.8mm, F.Cu at (-37.5, 25.7)
- added D10: RCLAMP0502B, Package_TO_SOT_SMD:SOT-416, F.Cu at (101.5, 7.75)
- added D11: RCLAMP0502B, Package_TO_SOT_SMD:SOT-416, F.Cu at (115.5, 7.75)
- added D12: RCLAMP0502B, Package_TO_SOT_SMD:SOT-416, F.Cu at (128.2, 7.75)
- added D13: RCLAMP0502B, Package_TO_SOT_SMD:SOT-416, F.Cu at (141.0, 7.75)
- added D14: RCLAMP0502B, Package_TO_SOT_SMD:SOT-416, F.Cu at (153.8, 7.75)
- added D2: PTVS5V0Z1USK, Diode_SMD:Nexperia_DSN1608-2_1.6x0.8mm, F.Cu at (-37.5, 28.1)
- added D2: LED, LED_SMD:LED_0603_1608Metric, F.Cu at (-53.3, 13.5)
- added D3: RCLAMP0502B, Package_TO_SOT_SMD:SOT-416, F.Cu at (11.0, 7.75)
- added D3: LED, LED_SMD:LED_0603_1608Metric, F.Cu at (-50.7, 13.5)
- added D4: LED, LED_SMD:LED_0603_1608Metric, F.Cu at (-48.1, 13.5)
- added D4: RCLAMP0502B, Package_TO_SOT_SMD:SOT-416, F.Cu at (23.8, 7.75)
- added D7: RCLAMP0502B, Package_TO_SOT_SMD:SOT-416, F.Cu at (63.2, 7.75)
- added D8: RCLAMP0502B, Package_TO_SOT_SMD:SOT-416, F.Cu at (76.0, 7.75)
- added D9: RCLAMP0502B, Package_TO_SOT_SMD:SOT-416, F.Cu at (88.8, 7.75)
- added DMX1: SM03B-SRSS-TB_LF__SN_, SamacSys_Parts:SM03BSRSSTBLFSN, F.Cu at (11.0, 2.50)
- added DMX10: SM03B-SRSS-TB_LF__SN_, SamacSys_Parts:SM03BSRSSTBLFSN, F.Cu at (128.2, 2.50)
- added DMX11: SM03B-SRSS-TB_LF__SN_, SamacSys_Parts:SM03BSRSSTBLFSN, F.Cu at (141.0, 2.50)
- added DMX12: SM03B-SRSS-TB_LF__SN_, SamacSys_Parts:SM03BSRSSTBLFSN, F.Cu at (153.8, 2.50)
- added DMX2: SM03B-SRSS-TB_LF__SN_, SamacSys_Parts:SM03BSRSSTBLFSN, F.Cu at (23.8, 2.50)
- added DMX3: SM03B-SRSS-TB_LF__SN_, SamacSys_Parts:SM03BSRSSTBLFSN, F.Cu at (36.5, 2.50)
- added DMX4: SM03B-SRSS-TB_LF__SN_, SamacSys_Parts:SM03BSRSSTBLFSN, F.Cu at (49.2, 2.50)
- added DMX5: SM03B-SRSS-TB_LF__SN_, SamacSys_Parts:SM03BSRSSTBLFSN, F.Cu at (63.2, 2.50)
- added DMX6: SM03B-SRSS-TB_LF__SN_, SamacSys_Parts:SM03BSRSSTBLFSN, F.Cu at (76.0, 2.50)
- added DMX7: SM03B-SRSS-TB_LF__SN_, SamacSys_Parts:SM03BSRSSTBLFSN, F.Cu at (88.8, 2.50)
- added DMX8: SM03B-SRSS-TB_LF__SN_, SamacSys_Parts:SM03BSRSSTBLFSN, F.Cu at (101.5, 2.50)
- added DMX9: SM03B-SRSS-TB_LF__SN_, SamacSys_Parts:SM03BSRSSTBLFSN, F.Cu at (115.5, 2.50)
- added IC10: 18024215401H, SamacSys_Parts:18024215401H, F.Cu at (87.5, 25.8)
- added IC11: 18024215401H, SamacSys_Parts:18024215401H, F.Cu at (100.2, 25.8)
- added IC12: 18024215401H, SamacSys_Parts:18024215401H, F.Cu at (114.2, 25.8)
- added IC13: 18024215401H, SamacSys_Parts:18024215401H, F.Cu at (127.0, 25.8)
- added IC14: 18024215401H, SamacSys_Parts:18024215401H, F.Cu at (139.8, 25.8)
- added IC15: 18024215401H, SamacSys_Parts:18024215401H, F.Cu at (152.5, 25.8)
- added IC16: TPP361063-T6TR, SamacSys_Parts:SOT95P280X95-6N, F.Cu at (-12.6, 10.2)
- added IC3: KTS1622EUAA-TR, SamacSys_Parts:QFN50P400X400X80-25N-D, F.Cu at (-39.5, 36.2)
- added IC4: 18024215401H, SamacSys_Parts:18024215401H, F.Cu at (9.75, 25.8)
- added IC5: 18024215401H, SamacSys_Parts:18024215401H, F.Cu at (22.5, 25.8)
- added IC6: 18024215401H, SamacSys_Parts:18024215401H, F.Cu at (35.2, 25.8)
- added IC7: 18024215401H, SamacSys_Parts:18024215401H, F.Cu at (48.0, 25.8)
- added IC8: 18024215401H, SamacSys_Parts:18024215401H, F.Cu at (62.0, 25.8)
- added IC9: 18024215401H, SamacSys_Parts:18024215401H, F.Cu at (74.8, 25.8)
- added R10: 10k, Resistor_SMD:R_0603_1608Metric, F.Cu at (-67.9, 17.5)
- added R10: R, Resistor_SMD:R_0603_1608Metric, F.Cu at (11.0, 10.0)
- added R21: R, Resistor_SMD:R_0603_1608Metric, F.Cu at (60.2, 10.0)
- added R22: R, Resistor_SMD:R_0603_1608Metric, F.Cu at (63.2, 10.0)
- added R23: R, Resistor_SMD:R_0603_1608Metric, F.Cu at (66.2, 10.0)
- added R24: R, Resistor_SMD:R_0603_1608Metric, F.Cu at (73.0, 10.0)
- added R25: R, Resistor_SMD:R_0603_1608Metric, F.Cu at (76.0, 10.0)
- added R26: R, Resistor_SMD:R_0603_1608Metric, F.Cu at (79.0, 10.0)
- added R27: R, Resistor_SMD:R_0603_1608Metric, F.Cu at (85.8, 10.0)
- added R28: R, Resistor_SMD:R_0603_1608Metric, F.Cu at (88.8, 10.0)
- added R29: R, Resistor_SMD:R_0603_1608Metric, F.Cu at (91.8, 10.0)
- added R30: R, Resistor_SMD:R_0603_1608Metric, F.Cu at (98.5, 10.0)
- added R31: R, Resistor_SMD:R_0603_1608Metric, F.Cu at (101.5, 10.0)
- added R32: R, Resistor_SMD:R_0603_1608Metric, F.Cu at (104.5, 10.0)
- added R33: R, Resistor_SMD:R_0603_1608Metric, F.Cu at (112.5, 10.0)
- added R34: R, Resistor_SMD:R_0603_1608Metric, F.Cu at (115.5, 10.0)
- added R35: R, Resistor_SMD:R_0603_1608Metric, F.Cu at (118.5, 10.0)
- added R36: R, Resistor_SMD:R_0603_1608Metric, F.Cu at (125.2, 10.0)
- added R37: R, Resistor_SMD:R_0603_1608Metric, F.Cu at (128.2, 10.0)
- added R38: R, Resistor_SMD:R_0603_1608Metric, F.Cu at (131.2, 10.0)
- added R39: R, Resistor_SMD:R_0603_1608Metric, F.Cu at (138.0, 10.0)
- added R40: R, Resistor_SMD:R_0603_1608Metric, F.Cu at (141.0, 10.0)
- added R41: R, Resistor_SMD:R_0603_1608Metric, F.Cu at (144.0, 10.0)
- added R42: R, Resistor_SMD:R_0603_1608Metric, F.Cu at (150.8, 10.0)
- added R43: R, Resistor_SMD:R_0603_1608Metric, F.Cu at (153.8, 10.0)
- added R44: R, Resistor_SMD:R_0603_1608Metric, F.Cu at (156.8, 10.0)
- added R7: 5k1, Resistor_SMD:R_0603_1608Metric, F.Cu at (-65.4, 17.5)
- added R7: 10k, Resistor_SMD:R_0603_1608Metric, F.Cu at (-75.4, 17.5)
- added R8: 10k, Resistor_SMD:R_0603_1608Metric, F.Cu at (-72.9, 17.5)
- added R8: 5k1, Resistor_SMD:R_0603_1608Metric, F.Cu at (-62.9, 17.5)
- added R9: R, Resistor_SMD:R_0603_1608Metric, F.Cu at (8.00, 10.0)
- added R9: 10k, Resistor_SMD:R_0603_1608Metric, F.Cu at (-70.4, 17.5)
- added SW2: SW_SPST, Button_Switch_SMD:SW_SPST_EVQP2, F.Cu at (-49.6, 7.38)
- added U10: ST485E, Package_SO:SOIC-8_3.9x4.9mm_P1.27mm, F.Cu at (128.2, 15.2)
- added U11: ST485E, Package_SO:SOIC-8_3.9x4.9mm_P1.27mm, F.Cu at (141.0, 15.2)
- added U12: ST485E, Package_SO:SOIC-8_3.9x4.9mm_P1.27mm, F.Cu at (153.8, 15.2)
- added U5: ST485E, Package_SO:SOIC-8_3.9x4.9mm_P1.27mm, F.Cu at (63.2, 15.2)
- added U6: ST485E, Package_SO:SOIC-8_3.9x4.9mm_P1.27mm, F.Cu at (76.0, 15.2)
- added U7: ST485E, Package_SO:SOIC-8_3.9x4.9mm_P1.27mm, F.Cu at (88.8, 15.2)
- added U8: ST485E, Package_SO:SOIC-8_3.9x4.9mm_P1.27mm, F.Cu at (101.5, 15.2)
- added U9: ST485E, Package_SO:SOIC-8_3.9x4.9mm_P1.27mm, F.Cu at (115.5, 15.2)
- C22: value 1n/2kV -> 0u1/6V3; footprint Capacitor_SMD:C_1206_3216Metric -> Capacitor_SMD:C_0603_1608Metric
- C23: value 1u/6V3 -> 0u1/6V3
- C24: value 1u/6V3 -> 1n/2kV; footprint Capacitor_SMD:C_0603_1608Metric -> Capacitor_SMD:C_1206_3216Metric
- C25, C26: value 1u/6V3 -> 10u/6V3
- moved USB1 115.8 mm to (-85.5, 40.0)
- moved IC2 100.7 mm to (50.0, 50.0), turned to 180 degrees
- moved SW1 84.4 mm to (-54.7, 7.38)
- moved C23 83.5 mm to (-72.9, 21.5), turned to 90 degrees
- moved C24 74.9 mm to (-49.3, 20.2), turned to 90 degrees
- moved IC1 71.0 mm to (34.8, 45.0)
- moved C25 52.0 mm to (5.50, 33.2)
- moved C22 49.0 mm to (-75.4, 21.5), turned to 90 degrees
- moved R6 40.7 mm to (-78.0, 17.5), turned to 90 degrees
- moved C20 35.8 mm to (-78.0, 21.5), turned to 90 degrees
- moved C26 34.0 mm to (6.50, 18.2)
- moved L1 28.6 mm to (-70.4, 21.5), turned to 90 degrees
- moved Y1 28.5 mm to (-53.8, 20.0), turned to 90 degrees
- moved C10 27.7 mm to (-78.0, 25.5), turned to 90 degrees
- moved R1 26.7 mm to (-67.9, 21.5), turned to 90 degrees
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Connections:
- C22 pad 1: GND -> 3V3
- C22 pad 2: Net-(USB1-SHIELD) -> GND
- C23 pad 1: /DMX_CH0/5V_DMX -> 3V3
- C23 pad 2: /DMX_CH0/GND_DMX -> GND
- C24 pad 1: /DMX_CH1/5V_DMX -> GND
- C24 pad 2: /DMX_CH1/GND_DMX -> Net-(USB1-SHIELD)
- C25 pad 1: /DMX_CH2/5V_DMX -> 5V0
- C25 pad 2: /DMX_CH2/GND_DMX -> GND
- C26 pad 1: /DMX_CH3/5V_DMX -> /DMX_CH0/5V_DMX
- C26 pad 2: /DMX_CH3/GND_DMX -> /DMX_CH0/GND_DMX
- IC2 pad 1: unconnected-(IC2-GPIO4-Pad1) -> /MCU/SPI_MISO
- IC2 pad 11: unconnected-(IC2-GPIO12-Pad11) -> /DMX0_TXD
- IC2 pad 12: unconnected-(IC2-GPIO13-Pad12) -> /DMX0_TXE
- IC2 pad 13: unconnected-(IC2-GPIO14-Pad13) -> /DMX0_RXD
- IC2 pad 14: unconnected-(IC2-GPIO15-Pad14) -> /DMX1_TXE
- IC2 pad 16: unconnected-(IC2-GPIO16-Pad16) -> /DMX1_TXD
- IC2 pad 17: unconnected-(IC2-GPIO17-Pad17) -> /DMX1_RXD
- IC2 pad 18: unconnected-(IC2-GPIO18-Pad18) -> /DMX2_TXD
- IC2 pad 19: unconnected-(IC2-GPIO19-Pad19) -> /DMX2_TXE
- IC2 pad 2: unconnected-(IC2-GPIO5-Pad2) -> /MCU/SPI_A0_DISP
- IC2 pad 20: unconnected-(IC2-GPIO20-Pad20) -> /DMX2_RXD
- IC2 pad 21: unconnected-(IC2-GPIO21-Pad21) -> /DMX3_TXD
- IC2 pad 22: unconnected-(IC2-GPIO22-Pad22) -> /DMX3_TXE
- IC2 pad 23: unconnected-(IC2-GPIO23-Pad23) -> /DMX3_RXD
- IC2 pad 25: unconnected-(IC2-GPIO24-Pad25) -> /DMX4_TXD
- IC2 pad 26: unconnected-(IC2-GPIO25-Pad26) -> /DMX4_TXE
- IC2 pad 27: unconnected-(IC2-GPIO26-Pad27) -> /DMX4_RXD
- IC2 pad 28: unconnected-(IC2-GPIO27-Pad28) -> /DMX5_TXD
- IC2 pad 3: unconnected-(IC2-GPIO6-Pad3) -> /MCU/ETH_INT
- IC2 pad 36: unconnected-(IC2-GPIO28-Pad36) -> /DMX5_TXE
- IC2 pad 37: unconnected-(IC2-GPIO29-Pad37) -> /DMX5_RXD
- IC2 pad 38: unconnected-(IC2-GPIO30-Pad38) -> /DMX6_TXD
- IC2 pad 39: unconnected-(IC2-GPIO31-Pad39) -> /DMX6_TXE
- IC2 pad 4: unconnected-(IC2-GPIO7-Pad4) -> /MCU/I2C_SCL
- IC2 pad 40: unconnected-(IC2-GPIO32-Pad40) -> /DMX6_RXD
- IC2 pad 42: unconnected-(IC2-GPIO33-Pad42) -> /DMX7_TXD
- IC2 pad 43: unconnected-(IC2-GPIO34-Pad43) -> /DMX7_TXE
- IC2 pad 44: unconnected-(IC2-GPIO35-Pad44) -> /DMX7_RXD
- IC2 pad 45: unconnected-(IC2-GPIO36-Pad45) -> /DMX8_TXD
- IC2 pad 46: unconnected-(IC2-GPIO37-Pad46) -> /DMX8_TXE
- IC2 pad 47: unconnected-(IC2-GPIO38-Pad47) -> /DMX8_RXD
- IC2 pad 48: unconnected-(IC2-GPIO39-Pad48) -> /DMX9_TXD
- IC2 pad 49: unconnected-(IC2-GPIO40_ADC0-Pad49) -> /DMX9_TXE
- IC2 pad 52: unconnected-(IC2-GPIO41_ADC1-Pad52) -> /DMX9_RXD
- IC2 pad 53: unconnected-(IC2-GPIO42_ADC2-Pad53) -> /DMX10_TXD
- IC2 pad 54: unconnected-(IC2-GPIO43_ADC3-Pad54) -> /DMX10_TXE
- IC2 pad 55: unconnected-(IC2-GPIO44_ADC4-Pad55) -> /DMX10_RXD
- IC2 pad 56: unconnected-(IC2-GPIO45_ADC5-Pad56) -> /DMX11_TXD
- IC2 pad 57: unconnected-(IC2-GPIO46_ADC6-Pad57) -> /DMX11_TXE
- IC2 pad 58: unconnected-(IC2-GPIO47_ADC7-Pad58) -> /DMX11_RXD
- IC2 pad 6: unconnected-(IC2-GPIO8-Pad6) -> /MCU/I2C_SDA
- IC2 pad 7: unconnected-(IC2-GPIO9-Pad7) -> /MCU/EXP_INT
- IC2 pad 77: unconnected-(IC2-GPIO0-Pad77) -> /MCU/SPI_CS_ETH
- IC2 pad 78: unconnected-(IC2-GPIO1-Pad78) -> /MCU/SPI_CS_DISP
- IC2 pad 79: unconnected-(IC2-GPIO2-Pad79) -> /MCU/SPI_SCLK
- IC2 pad 8: unconnected-(IC2-GPIO10-Pad8) -> /MCU/DEV_RST
- IC2 pad 80: unconnected-(IC2-GPIO3-Pad80) -> /MCU/SPI_MOSI
- IC2 pad 9: unconnected-(IC2-GPIO11-Pad9) -> /MCU/NEO_PIXEL
- U1 pad 2: /DMX_CH0/RE_5V -> /DMX_CH0/GND_DMX
- U1 pad 5: unconnected-(U1-GND-Pad5) -> /DMX_CH0/GND_DMX
- U1 pad 8: unconnected-(U1-VCC-Pad8) -> /DMX_CH0/5V_DMX
- U2 pad 2: /DMX_CH1/RE_5V -> /DMX_CH1/GND_DMX
- U2 pad 5: unconnected-(U2-GND-Pad5) -> /DMX_CH1/GND_DMX
- U2 pad 8: unconnected-(U2-VCC-Pad8) -> /DMX_CH1/5V_DMX
- U3 pad 2: /DMX_CH2/RE_5V -> /DMX_CH2/GND_DMX
- U3 pad 5: unconnected-(U3-GND-Pad5) -> /DMX_CH2/GND_DMX
- U3 pad 8: unconnected-(U3-VCC-Pad8) -> /DMX_CH2/5V_DMX
- U4 pad 2: /DMX_CH3/RE_5V -> /DMX_CH3/GND_DMX
- U4 pad 5: unconnected-(U4-GND-Pad5) -> /DMX_CH3/GND_DMX
- U4 pad 8: unconnected-(U4-VCC-Pad8) -> /DMX_CH3/5V_DMX
Routing:
- net (no net): vias 4 -> 6
Other:
- board size 100 x 100 mm -> 165 x 60 mm
