File: hw_v1/ArtNetNode.kicad_sch (KiCad schematic)
At the start: 0 parts

Commit message: started hardware
Other:
- added sheet DMX_CH10 (Schematics/DMX_Interface.kicad_sch)
- added sheet DMX_CH11 (Schematics/DMX_Interface.kicad_sch)
- added sheet DMX_CH4 (Schematics/DMX_Interface.kicad_sch)
- added sheet DMX_CH5 (Schematics/DMX_Interface.kicad_sch)
- added sheet DMX_CH6 (Schematics/DMX_Interface.kicad_sch)
- added sheet DMX_CH7 (Schematics/DMX_Interface.kicad_sch)
- added sheet DMX_CH8 (Schematics/DMX_Interface.kicad_sch)
- added sheet DMX_CH9 (Schematics/DMX_Interface.kicad_sch)
- added sheet Supply (Schematics/Supply.kicad_sch)
- sheet DMX_CH0 ports: added RXD, TXD, TXE; removed RX_D, RX_E, TX_D, TX_E
- sheet DMX_CH1 ports: added RXD, TXD, TXE; removed RX_D, RX_E, TX_D, TX_E
- sheet DMX_CH2 ports: added RXD, TXD, TXE; removed RX_D, RX_E, TX_D, TX_E
- sheet DMX_CH3 ports: added RXD, TXD, TXE; removed RX_D, RX_E, TX_D, TX_E
- sheet MCU ports: added DEV_RST, DISP_LED, DMX0_RXD, DMX0_TXD, DMX0_TXE, DMX10_RXD, DMX10_TXD, DMX10_TXE, DMX11_RXD, DMX11_TXD, DMX11_TXE, DMX1_RXD, DMX1_TXD, DMX1_TXE, DMX2_RXD, DMX2_TXD, DMX2_TXE, DMX3_RXD, DMX3_TXD, DMX3_TXE, DMX4_RXD, DMX4_TXD, DMX4_TXE, DMX5_RXD, DMX5_TXD, DMX5_TXE, DMX6_RXD, DMX6_TXD, DMX6_TXE, DMX7_RXD, DMX7_TXD, DMX7_TXE, DMX8_RXD, DMX8_TXD, DMX8_TXE, DMX9_RXD, DMX9_TXD, DMX9_TXE, ENC_A, ENC_B, ENC_SW, ETH_INT, NEO_PIXEL, SPI_A0_DISP, SPI_CS_DISP, SPI_CS_ETH, SPI_MISO, SPI_MOSI, SPI_SCLK; removed none
