File: hw_v1/Schematics/DMX_Interface.kicad_sch (KiCad schematic)
At the start: 7 parts, among them J2 SM03B-SRSS-TB_LF__SN_, U1 ST485E

Commit message: started hardware
Parts:
- added C25: 10u/6V3, Capacitor_SMD:C_0603_1608Metric, symbol Device:C
- added C27: 1u/6V3, Capacitor_SMD:C_0603_1608Metric, symbol Device:C
- added IC4: 18024215401H, SamacSys_Parts:18024215401H, symbol SamacSys_Parts:18024215401H
- C26: renamed from C23; value 1u/6V3 -> 10u/6V3
- renumbered J2 to DMX1
Connections:
- net RE_5V is gone; now on net GND_DMX: U1.2 (~{RE})
- net 5V_DMX: now also U1.8 (VCC), C27.1, IC4.10 (SEL), IC4.16 (VOUT)
- net DE_5V: now also IC4.14 (OUTA)
- net DI_5V: now also IC4.13 (OUTB)
- net DMX_N: now also DMX1.1; no longer DMX1.3
- net DMX_P: now also DMX1.3; no longer DMX1.1
- net GND_DMX: now also U1.5 (GND), C27.2, IC4.15 (GND2_1), IC4.9 (GND2_2)
- net RO_5V: now also IC4.12 (INC)
- new net 5V0: C25.1, IC4.1 (VCC)
- new net GND: C25.2, IC4.2 (GND1_1), IC4.8 (GND1_2)
- new net RXD: IC4.5 (OUTC)
- new net TXD: IC4.4 (INB)
- new net TXE: IC4.3 (INA)
Other:
- note added: "BUS-DRIVER"
- note added: "ISOLATOR + SUPPLY"
- note added: "TERMINATION + BIAS"
- moved on the sheet: C26, D3, DMX1, R10, R11, R9, U1
