File: hw_v1/Schematics/RP2350B.kicad_sch (KiCad schematic)
At the start: 39 parts, among them IC1 W25Q16JVSNIQ, IC2 RP2350B, J1 Conn_ARM_SWD_TagConnect_TC203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, SW1 SW_SPST, Y1 SiT1602AC-13-33E-12.000000

Commit message: started hardware
Parts:
- added C19, C21: 0u1/6V3, Capacitor_SMD:C_0603_1608Metric, symbol Device:C
- added IC3: KTS1622EUAA-TR, QFN50P400X400X80-25N-D, symbol SamacSys_Parts:KTS1622EUAA-TR
- added SW2: SW_SPST, Button_Switch_SMD:SW_SPST_EVQP2, symbol Switch:SW_SPST
- renumbered C19 to C20, C20 to C22, C21 to C23, C22 to C24
Connections:
- net 3V3: now also C19.1, C21.1, IC3.21 (VDD_P), IC3.23 (VDD_I2C)
- net GND: now also C19.2, C21.2, IC3.9 (GND), SW2.1 (A)
- net RUN: now also SW2.2 (B)
- net SPI_MISO: now reaches IC2.1 (GPIO4)
- net DMX0_TXD: now reaches IC2.11 (GPIO12)
- net DMX0_TXE: now reaches IC2.12 (GPIO13)
- net DMX0_RXD: now reaches IC2.13 (GPIO14)
- net DMX1_TXD: now reaches IC2.14 (GPIO15)
- net DMX1_TXE: now reaches IC2.16 (GPIO16)
- net DMX1_RXD: now reaches IC2.17 (GPIO17)
- net DMX2_TXD: now reaches IC2.18 (GPIO18)
- net DMX2_TXE: now reaches IC2.19 (GPIO19)
- net SPI_A0_DISP: now reaches IC2.2 (GPIO5)
- net DMX2_RXD: now reaches IC2.20 (GPIO20)
- net DMX3_TXD: now reaches IC2.21 (GPIO21)
- net DMX3_TXE: now reaches IC2.22 (GPIO22)
- net DMX3_RXD: now reaches IC2.23 (GPIO23)
- net DMX4_TXD: now reaches IC2.25 (GPIO24)
- net DMX4_TXE: now reaches IC2.26 (GPIO25)
- net DMX4_RXD: now reaches IC2.27 (GPIO26)
- net DMX5_TXD: now reaches IC2.28 (GPIO27)
- net ETH_INT: now reaches IC2.3 (GPIO6)
- net DMX5_TXE: now reaches IC2.36 (GPIO28)
- net DMX5_RXD: now reaches IC2.37 (GPIO29)
- net DMX6_TXD: now reaches IC2.38 (GPIO30)
- net DMX6_TXE: now reaches IC2.39 (GPIO31)
- net I2C_SCL: now reaches IC2.4 (GPIO7)
- net I2C_SCL: now also IC3.19 (SCL)
- net DMX6_RXD: now reaches IC2.40 (GPIO32)
- net DMX7_TXD: now reaches IC2.42 (GPIO33)
- net DMX7_TXE: now reaches IC2.43 (GPIO34)
- net DMX7_RXD: now reaches IC2.44 (GPIO35)
- net DMX8_TXD: now reaches IC2.45 (GPIO36)
- net DMX8_TXE: now reaches IC2.46 (GPIO37)
- net DMX8_RXD: now reaches IC2.47 (GPIO38)
- net DMX9_TXD: now reaches IC2.48 (GPIO39)
- net DMX9_TXE: now reaches IC2.49 (GPIO40_ADC0)
- net DMX9_RXD: now reaches IC2.52 (GPIO41_ADC1)
- net DMX10_TXD: now reaches IC2.53 (GPIO42_ADC2)
- net DMX10_TXE: now reaches IC2.54 (GPIO43_ADC3)
- net DMX10_RXD: now reaches IC2.55 (GPIO44_ADC4)
- net DMX11_TXD: now reaches IC2.56 (GPIO45_ADC5)
- net DMX11_TXE: now reaches IC2.57 (GPIO46_ADC6)
- net DMX11_RXD: now reaches IC2.58 (GPIO47_ADC7)
- net I2C_SDA: now reaches IC2.6 (GPIO8)
- net I2C_SDA: now also IC3.20 (SDA)
- net EXP_INT: now reaches IC2.7 (GPIO9)
- net EXP_INT: now also IC3.22 (~{INT})
- net SPI_CS_ETH: now reaches IC2.77 (GPIO0)
- net SPI_CS_DISP: now reaches IC2.78 (GPIO1)
- net SPI_SCLK: now reaches IC2.79 (GPIO2)
- net DEV_RST: now reaches IC2.8 (GPIO10)
- net DEV_RST: now also IC3.24 (~{RESET})
- net SPI_MOSI: now reaches IC2.80 (GPIO3)
- net NEO_PIXEL: now reaches IC2.9 (GPIO11)
- new net DISP_LED: IC3.10 (P1_0)
- new net ENC_A: IC3.1 (P0_0)
- new net ENC_B: IC3.2 (P0_1)
- new net ENC_SW: IC3.3 (P0_2)
